Commit message: add cylinder and piston joint in joint publisher

File: src/collaborative-robotic-sanding/abb_irb6700_support/urdf/irb6700_200_260_macro.xacro (robot description, xacro)
@@ -322,4 +322,24 @@
 		</joint>
 		<actuator name="joint_6_motor">
+		    <hardwareInterface>hardware_interface/EffortJointInterface</hardwareInterface>
+		    <mechanicalReduction>1</mechanicalReduction>
+		</actuator>
+	</transmission>
+	<transmission name="trans_piston_joint">
+		<type>transmission_interface/SimpleTransmission</type>
+		<joint name="${prefix}piston_joint">
+		    <hardwareInterface>hardware_interface/EffortJointInterface</hardwareInterface>
+		</joint>
+		<actuator name="piston_joint_motor">
+		    <hardwareInterface>hardware_interface/EffortJointInterface</hardwareInterface>
+		    <mechanicalReduction>1</mechanicalReduction>
+		</actuator>
+	</transmission>
+	<transmission name="trans_cylinder_joint">
+		<type>transmission_interface/SimpleTransmission</type>
+		<joint name="${prefix}cylinder_joint">
+		    <hardwareInterface>hardware_interface/EffortJointInterface</hardwareInterface>
+		</joint>
+		<actuator name="cylinder_joint_motor">
 		    <hardwareInterface>hardware_interface/EffortJointInterface</hardwareInterface>
 		    <mechanicalReduction>1</mechanicalReduction>
@@ -412,4 +432,6 @@
           <joint_name>${prefix}joint_5</joint_name>
           <joint_name>${prefix}joint_6</joint_name>
+		  <joint_name>${prefix}cylinder_joint</joint_name>
+          <joint_name>${prefix}piston_joint</joint_name>
         </plugin>
         <plugin name='crs_gazebo_plugins_joint_pose_trajectory' filename='libcrs_gazebo_plugins_joint_pose_trajectory.so'>

Commit message: added inertial tags to abb robot links

File: src/collaborative-robotic-sanding/abb_irb6700_support/urdf/irb6700_200_260_macro.xacro (robot description, xacro)
@@ -25,4 +25,9 @@
         <xacro:material_abb_yellow/>
       </collision>
+      <inertial>
+        <mass value="12.93"/>
+        <origin rpy="0 1.57079632679 0" xyz="-0.3059856723 0.0 0.175"/>
+        <inertia ixx="0.421716012238" ixy="0.0" ixz="0.0" iyy="0.421716012238" iyz="0.0" izz="0.036365625"/>
+      </inertial>
     </link>
     <link name="${prefix}link_1">
@@ -41,4 +46,9 @@
         <xacro:material_abb_yellow/>
       </collision>
+      <inertial>
+        <mass value="12.93"/>
+        <origin rpy="0 1.57079632679 0" xyz="-0.3059856723 0.0 0.175"/>
+        <inertia ixx="0.421716012238" ixy="0.0" ixz="0.0" iyy="0.421716012238" iyz="0.0" izz="0.036365625"/>
+      </inertial>
     </link>
     <link name="${prefix}cylinder">
@@ -57,4 +67,9 @@
         <xacro:material_abb_yellow/>
       </collision>
+      <inertial>
+        <mass value="12.93"/>
+        <origin rpy="0 1.57079632679 0" xyz="-0.3059856723 0.0 0.175"/>
+        <inertia ixx="0.421716012238" ixy="0.0" ixz="0.0" iyy="0.421716012238" iyz="0.0" izz="0.036365625"/>
+      </inertial>
     </link>
     <link name="${prefix}piston">
@@ -73,4 +88,9 @@
         <xacro:material_abb_yellow/>
       </collision>
+      <inertial>
+        <mass value="12.93"/>
+        <origin rpy="0 1.57079632679 0" xyz="-0.3059856723 0.0 0.175"/>
+        <inertia ixx="0.421716012238" ixy="0.0" ixz="0.0" iyy="0.421716012238" iyz="0.0" izz="0.036365625"/>
+      </inertial>
     </link>
     <link name="${prefix}link_2">
@@ -89,4 +109,9 @@
         <xacro:material_abb_yellow/>
       </collision>
+      <inertial>
+        <mass value="12.93"/>
+        <origin rpy="0 1.57079632679 0" xyz="-0.3059856723 0.0 0.175"/>
+        <inertia ixx="0.421716012238" ixy="0.0" ixz="0.0" iyy="0.421716012238" iyz="0.0" izz="0.036365625"/>
+      </inertial>
     </link>
     <link name="${prefix}link_3">
@@ -105,4 +130,9 @@
         <xacro:material_abb_yellow/>
       </collision>
+      <inertial>
+        <mass value="12.93"/>
+        <origin rpy="0 1.57079632679 0" xyz="-0.3059856723 0.0 0.175"/>
+        <inertia ixx="0.421716012238" ixy="0.0" ixz="0.0" iyy="0.421716012238" iyz="0.0" izz="0.036365625"/>
+      </inertial>
     </link>
     <link name="${prefix}link_4">
@@ -121,4 +151,9 @@
         <xacro:material_abb_yellow/>
       </collision>
+      <inertial>
+        <mass value="12.93"/>
+        <origin rpy="0 1.57079632679 0" xyz="-0.3059856723 0.0 0.175"/>
+        <inertia ixx="0.421716012238" ixy="0.0" ixz="0.0" iyy="0.421716012238" iyz="0.0" izz="0.036365625"/>
+      </inertial>
     </link>
     <link name="${prefix}link_5">
@@ -137,4 +172,9 @@
         <xacro:material_abb_yellow/>
       </collision>
+      <inertial>
+        <mass value="12.93"/>
+        <origin rpy="0 1.57079632679 0" xyz="-0.3059856723 0.0 0.175"/>
+        <inertia ixx="0.421716012238" ixy="0.0" ixz="0.0" iyy="0.421716012238" iyz="0.0" izz="0.036365625"/>
+      </inertial>
     </link>
     <link name="${prefix}link_6">
@@ -153,4 +193,9 @@
         <xacro:material_abb_yellow/>
       </collision>
+      <inertial>
+        <mass value="12.93"/>
+        <origin rpy="0 1.57079632679 0" xyz="-0.3059856723 0.0 0.175"/>
+        <inertia ixx="0.421716012238" ixy="0.0" ixz="0.0" iyy="0.421716012238" iyz="0.0" izz="0.036365625"/>
+      </inertial>
     </link>
     <!--add e-e-->
@@ -181,4 +226,5 @@
       <axis xyz="0 0 1" />
       <limit lower="-${radians(170)}" upper="${radians(170)}" effort="0" velocity="${radians(110)}" />
+      <dynamics damping="0.0" friction="0.0"/>
     </joint>
     <joint name="${prefix}joint_2" type="revolute">
@@ -188,4 +234,5 @@
       <axis xyz="0 1 0" />
       <limit lower="-${radians(65)}" upper="${radians(85)}" effort="0" velocity="${radians(110)}" />
+      <dynamics damping="0.0" friction="0.0"/>
     </joint>
     <joint name="${prefix}joint_3" type="revolute">
@@ -195,4 +242,5 @@
       <axis xyz="0 1 0" />
       <limit lower="-${radians(180)}" upper="${radians(70)}" effort="0" velocity="${radians(110)}" />
+      <dynamics damping="0.0" friction="0.0"/>
     </joint>
     <joint name="${prefix}joint_4" type="revolute">
@@ -202,4 +250,5 @@
       <axis xyz="1 0 0" />
       <limit lower="-${radians(300)}" upper="${radians(300)}" effort="0" velocity="${radians(190)}" />
+      <dynamics damping="0.0" friction="0.0"/>
     </joint>
     <joint name="${prefix}joint_5" type="revolute">
@@ -209,4 +258,5 @@
       <axis xyz="0 1 0" />
       <limit lower="-${radians(130)}" upper="${radians(130)}" effort="0" velocity="${radians(150)}" />
+      <dynamics damping="0.0" friction="0.0"/>
     </joint>
     <joint name="${prefix}joint_6" type="revolute">
@@ -216,6 +266,7 @@
       <axis xyz="1 0 0" />
       <limit lower="-${radians(360)}" upper="${radians(360)}" effort="0" velocity="${radians(210)}" />
-    </joint>
-    <joint name="${prefix}cylinder_joint" type="revolute">
+      <dynamics damping="0.0" friction="0.0"/>
+    </joint>
+    <joint name="${prefix}cylinder_joint" type="fixed">
       <origin xyz="-0.349 -0.194 -0.142" rpy="0 0 0" />
       <parent link="${prefix}link_1" />
@@ -225,5 +276,5 @@
       <limit lower="-${radians(65*0.25)}" upper="${radians(85*0.25)}" effort="0" velocity="100" />
     </joint>
-    <joint name="${prefix}piston_joint" type="prismatic">
+    <joint name="${prefix}piston_joint" type="fixed">
       <origin xyz="0 0 0" rpy="0.20897 0 -${radians(90)}" />
       <parent link="${prefix}cylinder" />
@@ -422,6 +473,6 @@
         <plugin name='gazebo_ros_joint_state_publisher' filename='libgazebo_ros_joint_state_publisher.so'>
           <ros>
-              <namespace>/test</namespace>
-              <argument>joint_states:=joint_states</argument>
+              <namespace>crs</namespace>
+              <argument>--ros-args --remap  joint_states:=${prefix}/joint_states</argument>
           </ros>
           <update_rate>50</update_rate>
@@ -432,11 +483,11 @@
           <joint_name>${prefix}joint_5</joint_name>
           <joint_name>${prefix}joint_6</joint_name>
-		  <joint_name>${prefix}cylinder_joint</joint_name>
-          <joint_name>${prefix}piston_joint</joint_name>
+		      <!--<joint_name>${prefix}cylinder_joint</joint_name>
+          <joint_name>${prefix}piston_joint</joint_name>-->
         </plugin>
         <plugin name='crs_gazebo_plugins_joint_pose_trajectory' filename='libcrs_gazebo_plugins_joint_pose_trajectory.so'>
             <ros>
               <namespace>sim</namespace>
-              <argument>follow_joint_trajectory:=${prefix}follow_joint_trajectory</argument>
+              <argument>--ros-args --remap follow_joint_trajectory:=${prefix}follow_joint_trajectory</argument>
             </ros>
             <update_rate>20</update_rate>
